Commit message: 抽取csv数据的position进行播放

File: install_aarch64/share/action_data_offset/urdf/CASBOT02_ENCOS_7dof_shell_20251015_P1L.urdf (robot description, URDF)
Before this commit: robot CB02_URDF(ECS)130C, 60 links, 59 joints
Joints:
- joint left_elbow_pitch_joint: limit lower=-2.268 upper=0 effort=75 velocity=12.2 -> lower=-2.268 upper=0.34 effort=75 velocity=12.2
- joint right_elbow_pitch_joint: limit lower=-2.268 upper=0 effort=75 velocity=12.2 -> lower=-2.268 upper=0.34 effort=75 velocity=12.2
